File: hexpansion.kicad_sch (KiCad schematic)
At the start: 7 parts, among them J1 Hexpansion-Connector, J2 Conn_02x10_Odd_Even

Commit message: first pass at sch
Parts:
- removed J2: Conn_02x10_Odd_Even, Connector_PinHeader_2.54mm:PinHeader_2x10_P2.54mm_Vertical, symbol Connector_Generic:Conn_02x10_Odd_Even
- removed R1: R, Resistor_SMD:R_0603_1608Metric, symbol Device:R
- added C1, C2: 4.7 uF, symbol Device:C_Small
- added C3: 0.1 uF, symbol Device:C_Small
- added D2, D3, D4: IR17-21C/TR8, symbol Device:LED
- added J2: Conn_ARM_SWD_TagConnect_TC2030, Connector:Tag-Connect_TC2030-IDC-FP_2x03_P1.27mm_Vertical, symbol Connector:Conn_ARM_SWD_TagConnect_TC2030
- added JP2, JP3, JP4: SolderJumper_2_Open, symbol Jumper:SolderJumper_2_Open
- added Q1, Q2, Q3, Q4: 2N7002, Package_TO_SOT_SMD:SOT-23, symbol Transistor_FET:2N7002
- added R1, R2, R4: 10k, symbol Device:R_Small
- added R10, R12, R6, R8: 1k, symbol Device:R_Small
- added R11, R3, R5, R7, R9: 100, symbol Device:R_Small
- added R13: DNL, symbol Device:R_Small
- added TP1, TP2: TestPoint, symbol Connector:TestPoint
- added TP10, TP3, TP4, TP5, TP6, TP7, TP8, TP9: TestPoint_Small, symbol Connector:TestPoint_Small
- added U1: ~, Package_DFN_QFN:QFN-16-1EP_3x3mm_P0.5mm_EP1.7x1.7mm, symbol parts:PY32F002AW15U
- added U2: ~, symbol parts:IRM-H6xxT
- D1: value LED -> IR17-21C/TR8; footprint LED_SMD:LED_0805_2012Metric -> (none)
Connections:
- net GND: now also C1.2, C2.2, C3.2, J2.5 (GND), Q1.2 (S), Q2.2 (S), Q3.2 (S), Q4.2 (S), U1.17 (GND), U2.1 (GND), U2.2 (GND); no longer D1.1 (K)
- net HS_F: now also JP2.1 (A)
- net HS_G: now also JP3.1 (A)
- net HS_H: now also JP4.1 (A)
- net SCL: now also R2.2, TP1.1, U1.9 (PA3)
- net SDA: now also R1.2, TP2.1, U1.8 (PA2)
- net at D1.2 (A): now also R5.2
- net 3V3 renamed +3.3V
- net +3.3V: now also C2.1, C3.1, J2.1 (VCC), R1.1, R11.1, R13.1, R2.1, R3.2, R4.1, R5.1, R7.1, R9.1, U1.15 (VCC)
- new net: TP7.1, U1.16 (PA8)
- new net: Q2.1 (G), R8.2
- new net: D2.1 (K), Q2.3 (D)
- new net: TP10.1, U1.1 (PB1)
- new net: TP4.1, U1.10 (PA4)
- new net: TP5.1, U1.11 (PA5)
- new net: TP6.1, U1.12 (PA6)
- new net: TP9.1, U1.14 (PB0)
- new net: TP8.1, U1.2 (PA12)
- new net: TP3.1, U1.7 (PA1)
- new net: Q4.1 (G), R12.2
- new net: D4.1 (K), Q4.3 (D)
- new net: D3.1 (K), Q3.3 (D)
- new net: D3.2 (A), R9.2
- new net: D2.2 (A), R7.2
- new net: Q3.1 (G), R10.2
- new net: C1.1, R3.1, U2.4 (Vcc)
- new net: D1.1 (K), Q1.3 (D)
- new net: D4.2 (A), R11.2
- new net: Q1.1 (G), R6.2
- new net IR_RX: R4.2, U1.6 (PA0), U2.3 (Vout)
- new net IR_TX: R10.1, R12.1, R6.1, R8.1, U1.13 (PA7)
- new net SWCLK: J2.4 (SWCLK), JP2.2 (B), U1.4 (PA14/SWC)
- new net SWDIO: J2.2 (SWDIO), JP3.2 (B), U1.3 (PA13/SWD)
- new net ~{RST}: J2.3 (~{RESET}), JP4.2 (B), R13.2, U1.5 (PF2/~{RST})
- no-connect marks 0 -> 1
Other:
- note added: "TIM1_CH3"
- note added: "Vf = 1 V - 1.5 V Assume typ Vf = 1.25 V target If = 20 mA R = (3.3 V - 1.25 V) / 20 mA = 102.5 Ohm ~= 100 Ohm If = 18 mA - 23 mA"
- note added: "legal use: TIM1_CH1N illegal use: TIM17_CH1 out?"
- moved on the sheet: J1
