File: hexpansion.kicad_pcb (KiCad board)
At the start: 2 copper layers, 32 x 36.6 mm, 44 parts, among them J1 Hexpansion-Connector, J2 Conn_ARM_SWD_TagConnect_TC2030, Q1 2N7002, Q2 2N7002, Q3 2N7002, Q4 2N7002, U1 PY32F002AW15U, U2 IRM-H638T/TR2

Commit message: some pcb doodles
Other:
- board text added: "2024 04-23"
- board text added: "IR Remote Tool Design by R"
Changed lines of the file:
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@@
+	)
+	(gr_line
+		(start 120.9 109.5)
+		(end 121.2 109.1)
+		(stroke
+			(width 0.15)
+			(type default)
+		)
+		(layer "B.SilkS")
+	)
+	(gr_line
+		(start 121.9 107.4)
+		(end 119.4 107.4)
+		(stroke
+			(width 0.15)
+			(type default)
+		)
+		(layer "B.SilkS")
+	)
+	(gr_line
+		(start 120.4 109.5)
+		(end 120.9 109.5)
+		(stroke
+			(width 0.15)
+			(type default)
+		)
+		(layer "B.SilkS")
+	)
+	(gr_line
+		(start 120.1 109.1)
+		(end 120.4 109.5)
+		(stroke
+			(width 0.15)
+			(type default)
+		)
+		(layer "B.SilkS")
+	)
+	(gr_line
+		(start 119.4 105.2)
+		(end 121.9 105.2)
+		(stroke
+			(width 0.15)
+			(type default)
+		)
+		(layer "B.SilkS")
+	)
+	(gr_line
+		(start 121 108.1)
+		(end 120.6 108.1)
+		(stroke
+			(width 0.15)
+			(type default)
+		)
+		(layer "B.SilkS")
+	)
+	(gr_line
+		(start 119.4 107.4)
+		(end 120.65 107)
+		(stroke
+			(width 0.15)
+			(type default)
+		)
+		(layer "B.SilkS")
+	)
+	(gr_line
+		(start 121 107.8)
+		(end 120.9 107.7)
+		(stroke
+			(width 0.15)
+			(type default)
+		)
+		(layer "B.SilkS")
+	)
+	(gr_line
+		(start 121 107.7)
+		(end 121 107.8)
+		(stroke
+			(width 0.15)
+			(type default)
+		)
+		(layer "B.SilkS")
+	)
+	(gr_line
+		(start 120.6 108.1)
+		(end 121 107.7)
+		(stroke
+			(width 0.15)
+			(type default)
+		)
+		(layer "B.SilkS")
+	)
+	(gr_line
+		(start 120.7 108.4)
+		(end 121 108.1)
+		(stroke
+			(width 0.15)
+			(type default)
+		)
+		(layer "B.SilkS")
+	)
+	(gr_line
+		(start 120.9 108.7)
+		(end 120.4 108.7)
+		(stroke
+			(width 0.15)
+			(type default)
+		)
+		(layer "B.SilkS")
+	)
+	(gr_line
+		(start 121.2 109.1)
+		(end 120.9 108.7)
+		(stroke
+			(width 0.15)
+			(type default)
+		)
+		(layer "B.SilkS")
+	)
+	(gr_line
+		(start 121.9 107)
+		(end 119.4 107)
+		(stroke
+			(width 0.15)
+			(type default)
+		)
+		(layer "B.SilkS")
+	)
+	(gr_line
+		(start 121.9 105.2)
+		(end 121.9 107)
+		(stroke
+			(width 0.15)
+			(type default)
+		)
+		(layer "B.SilkS")
+	)
+	(gr_line
+		(start 119.4 107)
+		(end 119.4 105.2)
+		(stroke
+			(width 0.15)
+			(type default)
+		)
+		(layer "B.SilkS")
+	)
+	(gr_line
+		(start 121.9 107.4)
+		(end 120.65 107)
+		(stroke
+			(width 0.15)
+			(type default)
+		)
+		(layer "B.SilkS")
+	)
+	(gr_line
+		(start 120.9 107.7)
+		(end 121 107.7)
+		(stroke
+			(width 0.15)
+			(type default)
+		)
+		(layer "B.SilkS")
+	)
+	(gr_line
+		(start 120.4 108.7)
+		(end 120.1 109.1)
+		(stroke
+			(width 0.15)
+			(type default)
+		)
+		(layer "B.SilkS")
 	)
 	(gr_line
@@
 		(layer "User.1")
 	)
+	(gr_text "2024\n04-23"
+		(at 105 93 0)
+		(layer "B.Cu")
+		(effects
+			(font
+				(size 0.8 0.8)
+				(thickness 0.2)
+				(bold yes)
+			)
+			(justify left bottom mirror)
+		)
+	)
+	(gr_text "IR Remote Tool\nDesign by R"
+		(at 128 105 270)
+		(layer "B.SilkS")
+		(effects
+			(font
+				(size 1 1)
+				(thickness 0.15)
+			)
+			(justify left bottom mirror)
+		)
+	)
 	(gr_text "You may expand the \nhexpansion in this area"
